Commit message: add camera

File: src/cartographer_ros/cartographer_ros/urdf/simBot.xacro (robot description, xacro)
@@ -3,3 +3,4 @@
     <xacro:include filename="xacro/car.xacro" />
     <xacro:include filename="xacro/laser.xacro" />
+    <xacro:include filename="xacro/camera.xacro" />
 </robot>

File: src/cartographer_ros/cartographer_ros/urdf/xacro/car.xacro (robot description, xacro)
@@ -1,6 +1,4 @@
-<!-- 根标签，必须声明 xmlns:xacro -->
 <robot name="my_base" xmlns:xacro="http://www.ros.org/wiki/xacro">
-    <!-- 封装变量、常量 -->
-    <!-- PI 值设置精度需要高一些，否则后续车轮翻转量计算时，可能会出现肉眼不能察觉的车轮倾斜，从而导致模型抖动 -->
+    <!-- PI 值设置 -->
     <xacro:property name="PI" value="3.1415926" />
     <!-- 宏:黑色设置 -->
@@ -10,8 +8,8 @@
     <!-- 底盘属性 -->
     <!-- <xacro:property name="base_footprint_radius" value="0.001" /> -->
-    <xacro:property name="base_link_length" value="0.44" /> <!-- base_link 长 -->
-    <xacro:property name="base_link_width" value="0.30" /> <!-- base_link 宽 -->
+    <xacro:property name="base_link_length" value="0.55" /> <!-- base_link 长 -->
+    <xacro:property name="base_link_width" value="0.44" /> <!-- base_link 宽 -->
     <xacro:property name="base_link_height" value="0.21" /> <!-- base_link 高 -->
-    <xacro:property name="earth_space" value="0.08" /> <!-- 底盘离地间距 -->
+    <xacro:property name="earth_space" value="0.09" /> <!-- 底盘离地间距 -->
     <!-- <link name="base_footprint">
         <visual>
@@ -26,5 +24,5 @@
                 <box size="${base_link_length} ${base_link_width} ${base_link_height}" />
             </geometry>
-            <origin xyz="0 0 0" rpy="0 0 0" />
+            <origin xyz="0 0 ${earth_space}" rpy="0 0 0" />
             <material name="yellow">
                 <color rgba="0.5 0.3 0.0 0.5" />
@@ -37,5 +35,5 @@
         <origin xyz="0 0 ${earth_space + base_link_height / 2 }" />
     </joint> -->
-    <!-- direction link -->
+    <!-- direction link 一个红色的圆盘指示小车车头的方向 -->
     <link name="dir_link">
         <visual>
@@ -51,5 +49,4 @@
     </joint>
     <!-- 驱动轮 -->
-    <!-- 驱动轮属性 -->
     <xacro:property name="wheel_radius" value="0.085" /> <!-- 半径 -->
     <xacro:property name="wheel_length" value="0.045" /> <!-- 宽度 -->
@@ -72,8 +69,7 @@
         </joint>
     </xacro:macro>
-    <xacro:add_wheels name="left" flag="1" />
-    <xacro:add_wheels name="right" flag="-1" />
+    <!-- <xacro:add_wheels name="left" flag="1" />
+    <xacro:add_wheels name="right" flag="-1" /> -->
     <!-- 支撑轮 -->
-    <!-- 支撑轮属性 -->
     <xacro:property name="support_wheel_radius" value="0.03" /> <!-- 支撑轮半径 -->
     <!-- 支撑轮宏 -->

File: src/cartographer_ros/cartographer_ros/urdf/xacro/laser.xacro (robot description, xacro)
@@ -3,7 +3,8 @@
         <color rgba="1.0 0.5 0.2 1" />
     </material>
-    <material name="gray">
-        <color rgba="0.2 0.2 0.2 1" />
+    <material name="green">
+        <color rgba="0.5 1.0 0.5 0.6" />
     </material>
+    <!-- IMU -->
     <link name="imu_link">
         <visual>
@@ -13,5 +14,5 @@
             <box size="0.0 0.0 0.0" />
         </geometry>
-        <material name="orange" />
+        <material name="green" />
         </visual>
     </link>
@@ -22,7 +23,8 @@
     </joint>
     <!-- 雷达 -->
-    <!-- 雷达属性 -->
     <xacro:property name="laser_length" value="0.0935" /> <!-- 高度 -->
     <xacro:property name="laser_radius" value="0.04447" /> <!-- 半径 -->
+    <xacro:property name="laser_x" value="0.445" /> <!-- x轴距离 -->
+    <xacro:property name="laser_y" value="0.345" /> <!-- y轴距离 -->
     <xacro:macro name="add_lasers" params="name flag">
         <link name="laser_wj${name}">
@@ -32,5 +34,5 @@
                 <cylinder length="${laser_length}" radius="${laser_radius}" />
             </geometry>
-            <material name="gray" />
+            <material name="green" />
             </visual>
         </link>
@@ -39,5 +41,5 @@
             <child link="laser_wj${name}" />
             <!-- y轴配准的话，2号laser y轴要多0.05 z=底盘高度/2+雷达高度/2 -->
-            <origin rpy="0 0 ${-(flag-1)*PI/2}" xyz="${flag*base_link_length/2} ${flag*base_link_width/2} ${base_link_height/2+earth_space/2}" />
+            <origin rpy="0 0 ${-(flag-1)*PI/2}" xyz="${flag*laser_x/2} ${flag*laser_y/2} ${base_link_height/2+earth_space+laser_length/2}" />
         </joint>
     </xacro:macro>
